File: hardware/kicad/r393c164_32x8/r393c164_32x8.kicad_pcb (KiCad board)
At the start: 2 copper layers, 143.5 x 50.8 mm, 67 parts, among them J1 Conn_01x05_Pin, J2 Conn_01x02_Pin, Q1 IRLML6401, Q2 IRLML6401, Q3 IRLML6401, Q4 IRLML6401, Q5 IRLML6401, Q6 IRLML6401, Q7 IRLML6401, Q8 IRLML6401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

Commit message: r393c164_32x8: fix defects in KiCad schematic / PCB
Parts:
- U1: value 74LS393 -> 74HC393
- U3, U5, U7, U9: value 74HC164 -> 74HC164 / CD54ACT164
Changed lines of the file:
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@@
 			)
 		)
-		(property "Value" "74HC164"
+		(property "Value" "74HC164 / CD54ACT164"
 			(at 0 5.28 90)
 			(layer "F.Fab")
@@
 			)
 		)
-		(property "Value" "74HC164"
+		(property "Value" "74HC164 / CD54ACT164"
 			(at 0 5.28 90)
 			(layer "F.Fab")
@@
 			)
 		)
-		(property "Value" "74LS393"
+		(property "Value" "74HC393"
 			(at 0 5.28 0)
 			(layer "F.Fab")
@@
 			)
 		)
-		(property "Value" "74HC164"
+		(property "Value" "74HC164 / CD54ACT164"
 			(at 0 5.28 90)
 			(layer "F.Fab")
@@
 			)
 		)
-		(property "Value" "74HC164"
+		(property "Value" "74HC164 / CD54ACT164"
 			(at 0 5.28 90)
 			(layer "F.Fab")
